File: hardware/Noise Meter.kicad_pcb (KiCad board)
At the start: 2 copper layers, 52 parts, among them J1 Conn_Coaxial, J2 Conn_01x05_Male, Q1 MMBT2222A, Q2 MMBT2222A, Q3 MMBT2222A, Q4 MMBT2222A, SW1 SW_DPST, U1 ISL28290, U2 LT6231, U3 AD8436, U4 PIC16F19156, U5 LCD-4-digit

Commit message: PCB V1.0
Parts:
- removed the C17 at (231.1, 38.1)
- removed the C18 at (241.3, 55.9)
- removed the U5 at (271.8, 74.9)
- added C1: 100uF, Capacitors_Tantalum_SMD:CP_Tantalum_Case-X_EIA-7343-43_Hand, F.Cu at (145.0, 61.0)
- added C10: 100uF, Capacitors_Tantalum_SMD:CP_Tantalum_Case-X_EIA-7343-43_Hand, F.Cu at (158.0, 85.0)
- added C2: 100uF, Capacitors_Tantalum_SMD:CP_Tantalum_Case-X_EIA-7343-43_Hand, F.Cu at (145.0, 67.0)
- added C27: 10uF, Capacitors_THT:C_Rect_L31.5mm_W13.0mm_P27.50mm_MKS4, F.Cu at (202.0, 95.5)
- added C28: 0.1uF, Capacitors_THT:C_Rect_L13.0mm_W6.0mm_P10.00mm_FKS3_FKP3_MKS4, F.Cu at (169.0, 75.5)
- added C29: 100uF, Capacitors_Tantalum_SMD:CP_Tantalum_Case-X_EIA-7343-43_Hand, F.Cu at (186.8, 85.2)
- added C3: 100uF, Capacitors_Tantalum_SMD:CP_Tantalum_Case-X_EIA-7343-43_Hand, F.Cu at (145.0, 73.0)
- added C31: 10uF, Capacitors_THT:C_Rect_L31.5mm_W13.0mm_P27.50mm_MKS4, F.Cu at (168.5, 95.5)
- added C33: 100nF, Capacitors_SMD:C_0603_HandSoldering, F.Cu at (167.8, 72.5)
- added C4: 100uF, Capacitors_Tantalum_SMD:CP_Tantalum_Case-X_EIA-7343-43_Hand, F.Cu at (145.0, 79.0)
- added C6: 100uF, Capacitors_Tantalum_SMD:CP_Tantalum_Case-X_EIA-7343-43_Hand, F.Cu at (158.0, 61.0)
- added C7: 100uF, Capacitors_Tantalum_SMD:CP_Tantalum_Case-X_EIA-7343-43_Hand, F.Cu at (158.0, 67.0)
- added C8: 100uF, Capacitors_Tantalum_SMD:CP_Tantalum_Case-X_EIA-7343-43_Hand, F.Cu at (158.0, 73.0)
- added CON1: LCD-4-digit, Noise Meter Kicad Footprint Library:4-digit-LCD-footprint, F.Cu at (169.0, 124.0)
- added CON2: 5110_LCD, Noise Meter Kicad Footprint Library:5110, B.Cu at (170.2, 130.0)
- added CON3: 5110_LCD_ALT, Noise Meter Kicad Footprint Library:5110-Alt, B.Cu at (191.0, 130.0)
- added J3: Conn_01x02, Pin_Headers:Pin_Header_Angled_1x02_Pitch2.54mm, F.Cu at (147.0, 112.5)
- added L1: FB, Inductors_SMD:L_0805, F.Cu at (201.1, 87.7)
- added L2: FB, Inductors_SMD:L_0805, F.Cu at (184.0, 79.5)
- added R1: 15K, Resistors_SMD:R_0603_HandSoldering, F.Cu at (184.2, 75.5)
- added R2: 82, Resistors_SMD:R_0603_HandSoldering, F.Cu at (168.4, 65.1)
- added REF**: Via dia 0.8mm drill 0.5mm, Noise Meter Kicad Footprint Library:Via-dia-0-8mm-drill-0-5mm, F.Cu at (206.0, 103.0)
- added REF**: Via dia 0.8mm drill 0.5mm, Noise Meter Kicad Footprint Library:Via-dia-0-8mm-drill-0-5mm, F.Cu at (206.0, 76.0)
- added REF**: Via dia 0.8mm drill 0.5mm, Noise Meter Kicad Footprint Library:Via-dia-0-8mm-drill-0-5mm, F.Cu at (206.0, 73.0)
- added REF**: Via dia 0.8mm drill 0.5mm, Noise Meter Kicad Footprint Library:Via-dia-0-8mm-drill-0-5mm, F.Cu at (206.0, 70.0)
- added REF**: Via dia 0.8mm drill 0.5mm, Noise Meter Kicad Footprint Library:Via-dia-0-8mm-drill-0-5mm, F.Cu at (206.0, 67.0)
- added REF**: Via dia 0.8mm drill 0.5mm, Noise Meter Kicad Footprint Library:Via-dia-0-8mm-drill-0-5mm, F.Cu at (206.0, 64.0)
- added REF**: Via dia 0.8mm drill 0.5mm, Noise Meter Kicad Footprint Library:Via-dia-0-8mm-drill-0-5mm, F.Cu at (206.0, 61.0)
- added REF**: Via dia 0.8mm drill 0.5mm, Noise Meter Kicad Footprint Library:Via-dia-0-8mm-drill-0-5mm, F.Cu at (206.0, 58.0)
- added REF**: Via dia 0.8mm drill 0.5mm, Noise Meter Kicad Footprint Library:Via-dia-0-8mm-drill-0-5mm, F.Cu at (137.0, 103.0)
- added REF**: Via dia 0.8mm drill 0.5mm, Noise Meter Kicad Footprint Library:Via-dia-0-8mm-drill-0-5mm, F.Cu at (151.0, 53.0)
- added REF**: Via dia 0.8mm drill 0.5mm, Noise Meter Kicad Footprint Library:Via-dia-0-8mm-drill-0-5mm, F.Cu at (166.0, 53.0)
- added REF**: Via dia 0.8mm drill 0.5mm, Noise Meter Kicad Footprint Library:Via-dia-0-8mm-drill-0-5mm, F.Cu at (206.0, 100.0)
- added REF**: Via dia 0.8mm drill 0.5mm, Noise Meter Kicad Footprint Library:Via-dia-0-8mm-drill-0-5mm, F.Cu at (184.0, 53.0)
- added REF**: Via dia 0.8mm drill 0.5mm, Noise Meter Kicad Footprint Library:Via-dia-0-8mm-drill-0-5mm, F.Cu at (205.0, 53.0)
- added REF**: Via dia 0.8mm drill 0.5mm, Noise Meter Kicad Footprint Library:Via-dia-0-8mm-drill-0-5mm, F.Cu at (187.0, 105.0)
- added REF**: Via dia 0.8mm drill 0.5mm, Noise Meter Kicad Footprint Library:Via-dia-0-8mm-drill-0-5mm, F.Cu at (137.0, 100.0)
- added REF**: Via dia 0.8mm drill 0.5mm, Noise Meter Kicad Footprint Library:Via-dia-0-8mm-drill-0-5mm, F.Cu at (154.0, 53.0)
- added REF**: Via dia 0.8mm drill 0.5mm, Noise Meter Kicad Footprint Library:Via-dia-0-8mm-drill-0-5mm, F.Cu at (169.0, 53.0)
- added REF**: Via dia 0.8mm drill 0.5mm, Noise Meter Kicad Footprint Library:Via-dia-0-8mm-drill-0-5mm, F.Cu at (181.0, 53.0)
- added REF**: Via dia 0.8mm drill 0.5mm, Noise Meter Kicad Footprint Library:Via-dia-0-8mm-drill-0-5mm, F.Cu at (202.0, 53.0)
- added REF**: Via dia 0.8mm drill 0.5mm, Noise Meter Kicad Footprint Library:Via-dia-0-8mm-drill-0-5mm, F.Cu at (190.0, 105.0)
- added REF**: Via dia 0.8mm drill 0.5mm, Noise Meter Kicad Footprint Library:Via-dia-0-8mm-drill-0-5mm, F.Cu at (137.0, 97.0)
- added REF**: Via dia 0.8mm drill 0.5mm, Noise Meter Kicad Footprint Library:Via-dia-0-8mm-drill-0-5mm, F.Cu at (206.0, 97.0)
- added REF**: Via dia 0.8mm drill 0.5mm, Noise Meter Kicad Footprint Library:Via-dia-0-8mm-drill-0-5mm, F.Cu at (139.0, 53.0)
- added REF**: Via dia 0.8mm drill 0.5mm, Noise Meter Kicad Footprint Library:Via-dia-0-8mm-drill-0-5mm, F.Cu at (163.0, 53.0)
- added REF**: Via dia 0.8mm drill 0.5mm, Noise Meter Kicad Footprint Library:Via-dia-0-8mm-drill-0-5mm, F.Cu at (178.0, 53.0)
- added REF**: Via dia 0.8mm drill 0.5mm, Noise Meter Kicad Footprint Library:Via-dia-0-8mm-drill-0-5mm, F.Cu at (199.0, 53.0)
- added REF**: Via dia 0.8mm drill 0.5mm, Noise Meter Kicad Footprint Library:Via-dia-0-8mm-drill-0-5mm, F.Cu at (193.0, 105.0)
- added REF**: Via dia 0.8mm drill 0.5mm, Noise Meter Kicad Footprint Library:Via-dia-0-8mm-drill-0-5mm, F.Cu at (137.0, 94.0)
- added REF**: Via dia 0.8mm drill 0.5mm, Noise Meter Kicad Footprint Library:Via-dia-0-8mm-drill-0-5mm, F.Cu at (137.0, 61.0)
- added REF**: Via dia 0.8mm drill 0.5mm, Noise Meter Kicad Footprint Library:Via-dia-0-8mm-drill-0-5mm, F.Cu at (157.0, 53.0)
- added REF**: Via dia 0.8mm drill 0.5mm, Noise Meter Kicad Footprint Library:Via-dia-0-8mm-drill-0-5mm, F.Cu at (175.0, 53.0)
- added REF**: Via dia 0.8mm drill 0.5mm, Noise Meter Kicad Footprint Library:Via-dia-0-8mm-drill-0-5mm, F.Cu at (196.0, 53.0)
- added REF**: Via dia 0.8mm drill 0.5mm, Noise Meter Kicad Footprint Library:Via-dia-0-8mm-drill-0-5mm, F.Cu at (206.0, 94.0)
- added REF**: Via dia 0.8mm drill 0.5mm, Noise Meter Kicad Footprint Library:Via-dia-0-8mm-drill-0-5mm, F.Cu at (196.0, 105.0)
- added REF**: Via dia 0.8mm drill 0.5mm, Noise Meter Kicad Footprint Library:Via-dia-0-8mm-drill-0-5mm, F.Cu at (137.0, 91.0)
- added REF**: Via dia 0.8mm drill 0.5mm, Noise Meter Kicad Footprint Library:Via-dia-0-8mm-drill-0-5mm, F.Cu at (137.0, 70.0)
- added REF**: Via dia 0.8mm drill 0.5mm, Noise Meter Kicad Footprint Library:Via-dia-0-8mm-drill-0-5mm, F.Cu at (142.0, 53.0)
- added REF**: Via dia 0.8mm drill 0.5mm, Noise Meter Kicad Footprint Library:Via-dia-0-8mm-drill-0-5mm, F.Cu at (172.0, 53.0)
- added REF**: Via dia 0.8mm drill 0.5mm, Noise Meter Kicad Footprint Library:Via-dia-0-8mm-drill-0-5mm, F.Cu at (193.0, 53.0)
- added REF**: Via dia 0.8mm drill 0.5mm, Noise Meter Kicad Footprint Library:Via-dia-0-8mm-drill-0-5mm, F.Cu at (199.0, 105.0)
- added REF**: Via dia 0.8mm drill 0.5mm, Noise Meter Kicad Footprint Library:Via-dia-0-8mm-drill-0-5mm, F.Cu at (181.0, 105.0)
- added REF**: Via dia 0.8mm drill 0.5mm, Noise Meter Kicad Footprint Library:Via-dia-0-8mm-drill-0-5mm, F.Cu at (137.0, 88.0)
- added REF**: Via dia 0.8mm drill 0.5mm, Noise Meter Kicad Footprint Library:Via-dia-0-8mm-drill-0-5mm, F.Cu at (137.0, 73.0)
- added REF**: Via dia 0.8mm drill 0.5mm, Noise Meter Kicad Footprint Library:Via-dia-0-8mm-drill-0-5mm, F.Cu at (206.0, 91.0)
- added REF**: Via dia 0.8mm drill 0.5mm, Noise Meter Kicad Footprint Library:Via-dia-0-8mm-drill-0-5mm, F.Cu at (137.0, 55.0)
- added REF**: Via dia 0.8mm drill 0.5mm, Noise Meter Kicad Footprint Library:Via-dia-0-8mm-drill-0-5mm, F.Cu at (160.0, 53.0)
- added REF**: Via dia 0.8mm drill 0.5mm, Noise Meter Kicad Footprint Library:Via-dia-0-8mm-drill-0-5mm, F.Cu at (190.0, 53.0)
- added REF**: Via dia 0.8mm drill 0.5mm, Noise Meter Kicad Footprint Library:Via-dia-0-8mm-drill-0-5mm, F.Cu at (202.0, 105.0)
- added REF**: Via dia 0.8mm drill 0.5mm, Noise Meter Kicad Footprint Library:Via-dia-0-8mm-drill-0-5mm, F.Cu at (175.0, 105.0)
- added REF**: Via dia 0.8mm drill 0.5mm, Noise Meter Kicad Footprint Library:Via-dia-0-8mm-drill-0-5mm, F.Cu at (137.0, 85.0)
- added REF**: Via dia 0.8mm drill 0.5mm, Noise Meter Kicad Footprint Library:Via-dia-0-8mm-drill-0-5mm, F.Cu at (137.0, 76.0)
- added REF**: Via dia 0.8mm drill 0.5mm, Noise Meter Kicad Footprint Library:Via-dia-0-8mm-drill-0-5mm, F.Cu at (137.0, 64.0)
- added REF**: Via dia 0.8mm drill 0.5mm, Noise Meter Kicad Footprint Library:Via-dia-0-8mm-drill-0-5mm, F.Cu at (145.0, 53.0)
- added REF**: Via dia 0.8mm drill 0.5mm, Noise Meter Kicad Footprint Library:Via-dia-0-8mm-drill-0-5mm, F.Cu at (187.0, 53.0)
- added REF**: Via dia 0.8mm drill 0.5mm, Noise Meter Kicad Footprint Library:Via-dia-0-8mm-drill-0-5mm, F.Cu at (206.0, 88.0)
- added REF**: Via dia 0.8mm drill 0.5mm, Noise Meter Kicad Footprint Library:Via-dia-0-8mm-drill-0-5mm, F.Cu at (205.0, 105.0)
- added REF**: Via dia 0.8mm drill 0.5mm, Noise Meter Kicad Footprint Library:Via-dia-0-8mm-drill-0-5mm, F.Cu at (169.0, 105.0)
- added REF**: Via dia 0.8mm drill 0.5mm, Noise Meter Kicad Footprint Library:Via-dia-0-8mm-drill-0-5mm, F.Cu at (137.0, 82.0)
- added REF**: Via dia 0.8mm drill 0.5mm, Noise Meter Kicad Footprint Library:Via-dia-0-8mm-drill-0-5mm, F.Cu at (137.0, 79.0)
- added REF**: Via dia 0.8mm drill 0.5mm, Noise Meter Kicad Footprint Library:Via-dia-0-8mm-drill-0-5mm, F.Cu at (137.0, 67.0)
- added REF**: Via dia 0.8mm drill 0.5mm, Noise Meter Kicad Footprint Library:Via-dia-0-8mm-drill-0-5mm, F.Cu at (137.0, 58.0)
- added REF**: Via dia 0.8mm drill 0.5mm, Noise Meter Kicad Footprint Library:Via-dia-0-8mm-drill-0-5mm, F.Cu at (148.0, 53.0)
- added REF**: Via dia 0.8mm drill 0.5mm, Noise Meter Kicad Footprint Library:Via-dia-0-8mm-drill-0-5mm, F.Cu at (206.0, 55.0)
- added REF**: Via dia 0.8mm drill 0.5mm, Noise Meter Kicad Footprint Library:Via-dia-0-8mm-drill-0-5mm, F.Cu at (184.0, 105.0)
- added REF**: Via dia 0.8mm drill 0.5mm, Noise Meter Kicad Footprint Library:Via-dia-0-8mm-drill-0-5mm, F.Cu at (138.0, 105.0)
- added REF**: Via dia 0.8mm drill 0.5mm, Noise Meter Kicad Footprint Library:Via-dia-0-8mm-drill-0-5mm, F.Cu at (206.0, 85.0)
- added REF**: Via dia 0.8mm drill 0.5mm, Noise Meter Kicad Footprint Library:Via-dia-0-8mm-drill-0-5mm, F.Cu at (141.0, 105.0)
- added REF**: Via dia 0.8mm drill 0.5mm, Noise Meter Kicad Footprint Library:Via-dia-0-8mm-drill-0-5mm, F.Cu at (144.0, 105.0)
- added REF**: Via dia 0.8mm drill 0.5mm, Noise Meter Kicad Footprint Library:Via-dia-0-8mm-drill-0-5mm, F.Cu at (150.0, 105.0)
- added REF**: Via dia 0.8mm drill 0.5mm, Noise Meter Kicad Footprint Library:Via-dia-0-8mm-drill-0-5mm, F.Cu at (162.0, 105.0)
- added REF**: Via dia 0.8mm drill 0.5mm, Noise Meter Kicad Footprint Library:Via-dia-0-8mm-drill-0-5mm, F.Cu at (159.0, 105.0)
- added REF**: Via dia 0.8mm drill 0.5mm, Noise Meter Kicad Footprint Library:Via-dia-0-8mm-drill-0-5mm, F.Cu at (156.0, 105.0)
- added REF**: Via dia 0.8mm drill 0.5mm, Noise Meter Kicad Footprint Library:Via-dia-0-8mm-drill-0-5mm, F.Cu at (147.0, 105.0)
- added REF**: Via dia 0.8mm drill 0.5mm, Noise Meter Kicad Footprint Library:Via-dia-0-8mm-drill-0-5mm, F.Cu at (153.0, 105.0)
- added REF**: Via dia 0.8mm drill 0.5mm, Noise Meter Kicad Footprint Library:Via-dia-0-8mm-drill-0-5mm, F.Cu at (206.0, 82.0)
- added REF**: Via dia 0.8mm drill 0.5mm, Noise Meter Kicad Footprint Library:Via-dia-0-8mm-drill-0-5mm, F.Cu at (206.0, 79.0)
- added SW2: SW_Push, Buttons_Switches_SMD:SW_SPST_B3SL-1002P, B.Cu at (201.5, 110.0)
- added SW3: SW_Push, Buttons_Switches_SMD:SW_SPST_B3SL-1002P, B.Cu at (201.5, 118.0)
- added SW4: SW_Push, Buttons_Switches_SMD:SW_SPST_B3SL-1002P, F.Cu at (201.5, 110.0)
- added SW5: SW_Push, Buttons_Switches_SMD:SW_SPST_B3SL-1002P, F.Cu at (201.5, 118.0)
- BT1, BT2: moved to B.Cu
- C14: value 100uF -> 10uF; footprint Capacitors_SMD:CP_Elec_6.3x7.7 -> Capacitors_SMD:CP_Elec_4x4.5
- C30: renamed from C21; value 22uF 20% 6.3V -> 0.1uF 20% 6.3V
- C5: footprint Capacitors_THT:C_Rect_L41.5mm_W24.0mm_P37.50mm_MKS4 -> Capacitors_Tantalum_SMD:CP_Tantalum_Case-X_EIA-7343-43_Hand
- C9: value 10uF -> 100uF; footprint Capacitors_THT:C_Rect_L26.5mm_W8.5mm_P22.50mm_MKS4 -> Capacitors_Tantalum_SMD:CP_Tantalum_Case-X_EIA-7343-43_Hand
- J1: footprint Connectors_Molex:Molex_SMA_Jack_Edge_Mount -> Noise Meter Kicad Footprint Library:SMA-CONN
- R3: renamed from R1; value 2.2K -> 510
- SW1: footprint Buttons_Switches_THT:SW_E-Switch_EG2219_DPDT_Angled -> Buttons_Switches_THT:SW_CuK_JS202011AQN_DPDT_Angled
- U1: value ISL28290 -> OPA2227EP
- U2: value LT6231 -> OPA2227EP
- moved J1 139.0 mm to (169.3, 58.1)
- moved J2 134.5 mm to (147.0, 130.1), turned to 180 degrees
- moved BT2 127.9 mm to (189.3, 72.0), turned to 0 degrees
- moved D1 117.1 mm to (150.2, 122.8), turned to 90 degrees
- moved R17 113.3 mm to (150.2, 127.7)
- moved C17 111.0 mm to (199.8, 69.2), turned to 0 degrees
- moved C18 106.8 mm to (195.2, 68.6), turned to 270 degrees
- moved C5 106.4 mm to (145.0, 85.0)
- moved U3 104.3 mm to (158.5, 120.2)
- moved SW1 102.8 mm to (201.7, 129.5)
- moved C19 101.6 mm to (201.1, 85.5), turned to 0 degrees
- moved C20 95.4 mm to (177.8, 74.8), turned to 0 degrees
- moved C32 94.6 mm to (165.0, 122.2), turned to 270 degrees
- moved BT1 91.6 mm to (153.7, 72.0), turned to 0 degrees
- moved C22 91.3 mm to (192.4, 80.4)
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- renumbered C13 to C12, C10 to C15, C12 to C16, C1 to C17, C3 to C18, C6 to C19, C2 to C20, C4 to C21, C7 to C22, C8 to C23, C20 to C24, C15 to C25, C16 to C26, C19 to C32, R5 to R10, R10 to R11, R14 to R12, R2 to R13, R4 to R14, R9 to R15, R13 to R16, R16 to R17, R15 to R18, R7 to R4, R8 to R5, R11 to R6, R12 to R7, R6 to R8, R3 to R9, U4 to U3, U3 to U5
Connections:
- C12 pad 1: Net-(C13-Pad1) -> Net-(C12-Pad1)
- C14 pad 1: Net-(C13-Pad1) -> Net-(C14-Pad1)
- C14 pad 2: Net-(C14-Pad2) -> Net-(C14-Pad1)
- C17 pad 1: +3V -> +3V_LNA
- C18 pad 1: +3V -> +3V_LNA
- C20 pad 2: -3V -> -3V_LNA
- C21 pad 2: -3V -> -3V_LNA
- C25 pad 2: GND -> +3V_Digital
- C25 pad 3: +3V -> GND
- C26 pad 2: GND -> -3V_Digital
- C26 pad 3: -3V -> GND
- C30 pad 1: Net-(C21-Pad1) -> Net-(C30-Pad1)
- C30 pad 2: GND -> Net-(C30-Pad2)
- C30 pad 3: Net-(C21-Pad3) -> GND
- C32 pad 1: +3V -> +3V_Digital
- C5 pad 1: Net-(C5-Pad1) -> Net-(C1-Pad1)
- C5 pad 2: Net-(C5-Pad2) -> Net-(C1-Pad2)
- C9 pad 1: Net-(C9-Pad1) -> Net-(C1-Pad1)
- C9 pad 2: GND -> Net-(C1-Pad2)
- D1 pad 2: +3V -> +3V_Digital
- J1 pad 1: Net-(C5-Pad1) -> Net-(C1-Pad1)
- J2 pad 2: +3V -> +3V_Digital
- Q1 pad 1: Net-(C5-Pad2) -> Net-(Q1-Pad1)
- Q2 pad 3: Net-(C5-Pad2) -> Net-(Q1-Pad1)
- Q3 pad 1: Net-(C5-Pad2) -> Net-(Q1-Pad1)
- Q4 pad 3: Net-(C5-Pad2) -> Net-(Q1-Pad1)
- R12 pad 1: Net-(C13-Pad1) -> Net-(C12-Pad1)
- R3 pad 1: Net-(C5-Pad2) -> Net-(C1-Pad2)
- R9 pad 1: Net-(R3-Pad1) -> Net-(C14-Pad1)
- SW1 pad 1: -3V -> (no net)
- SW1 pad 2: Net-(BT2-Pad2) -> +3V_Digital
- SW1 pad 3: +3V -> Net-(BT1-Pad1)
- SW1 pad 4: Net-(BT1-Pad1) -> (no net)
- SW1 pad 5: (no net) -> -3V_Digital
- SW1 pad 6: (no net) -> Net-(BT2-Pad2)
- U1 pad 1: Net-(R3-Pad1) -> Net-(C14-Pad1)
- U1 pad 3: Net-(C5-Pad2) -> Net-(Q1-Pad1)
- U1 pad 4: -3V -> -3V_LNA
- U1 pad 5: Net-(R3-Pad1) -> Net-(C14-Pad1)
- U1 pad 8: +3V -> +3V_LNA
- U2 pad 7: Net-(C13-Pad1) -> Net-(C12-Pad1)
- U3 pad 10: Net-(U4-Pad10) -> Net-(C30-Pad1)
- U3 pad 13: Net-(C21-Pad1) -> Net-(CON2-Pad3)
- U3 pad 20: +3V -> +3V_Digital
- U5 pad 10: Net-(C9-Pad1) -> Net-(C31-Pad1)
- U5 pad 13: Net-(C9-Pad1) -> Net-(C31-Pad1)
- U5 pad 14: Net-(C21-Pad3) -> Net-(C30-Pad2)
- U5 pad 15: Net-(C21-Pad3) -> Net-(C30-Pad2)
- U5 pad 3: Net-(C14-Pad2) -> Net-(C29-Pad2)
Routing:
- net GND: track 0.00 -> 286.7 mm, vias 0 -> 24
- net +3V_Digital: track 0.00 -> 160.0 mm
- net Net-(BT1-Pad1): track 0.00 -> 137.1 mm
- net -3V_Digital: track 0.00 -> 126.5 mm
- net +3V: track 0.00 -> 124.9 mm, vias 0 -> 2
- net Net-(C1-Pad1): track 0.00 -> 81.7 mm
- net Net-(C1-Pad2): track 0.00 -> 72.9 mm
- net -3V: track 0.00 -> 72.7 mm
- net Net-(SW2-Pad2): track 0.00 -> 67.1 mm, vias 0 -> 2
- net Net-(SW3-Pad2): track 0.00 -> 65.6 mm, vias 0 -> 2
- net Net-(CON1-Pad6): track 0.00 -> 60.2 mm
- net Net-(BT2-Pad2): track 0.00 -> 56.2 mm
- net Net-(CON1-Pad5): track 0.00 -> 55.8 mm
- net Net-(CON1-Pad12): track 0.00 -> 49.8 mm
- net Net-(CON1-Pad9): track 0.00 -> 47.8 mm
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- added copper zone on B.Cu, net GND
Other:
- board outline added: 73 x 81 mm
- net class 3V_Digital added: clearance 0.2, trace_width 0.45, via_dia 0.8, via_drill 0.6
- net class ground added: clearance 0.25, trace_width 0.5, via_dia 0.6, via_drill 0.4
