File: hardware/Noise Meter.kicad_pcb (KiCad board)
At the start: 2 copper layers, 73 x 81 mm, 151 parts, among them CON1 LCD-4-digit, CON2 5110_LCD, CON3 5110_LCD_ALT, J1 Conn_Coaxial, J2 Conn_01x05_Male, J3 Conn_01x02, Q1 MMBT2222A, Q2 MMBT2222A, Q3 MMBT2222A, Q4 MMBT2222A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

Commit message: final touch ups and gerber files added
Parts:
- moved BT1 1.00 mm to (153.7, 71.0)
- moved BT2 1.00 mm to (189.3, 71.0)
- moved C28 0.50 mm to (169.0, 76.0)
Connections:
- net Net-(C30-Pad1) renamed /Vrms
Routing:
- net Net-(C14-Pad1): track 25.4 -> 31.5 mm
- net -3V: track 72.7 -> 74.3 mm
- net Net-(C27-Pad2): track 10.4 -> 9.25 mm
- net Net-(BT2-Pad2): track 56.2 -> 57.3 mm
- net Net-(BT1-Pad1): track 137.1 -> 138.3 mm
- net GND: track 286.7 -> 285.7 mm
- net /Vrms: track 40.4 -> 41.0 mm
Other:
- board text added: "2018"
- board text added: "CC"
- board text added: "GND"
- board text added: "ICSPCLK"
- board text added: "ICSPDAT"
- board text added: "VDD"
- board text added: "VPP"
- board text added: "Vrms"

Commit message: first pcb fabrication version
Other:
- board text added: "V1.0"
Changed lines of the file:
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@@
     (area 126.392858 49.435 216.607143 133.665)
     (thickness 1.6)
-    (drawings 21)
-    (tracks 619)
+    (drawings 22)
+    (tracks 620)
     (zones 0)
     (modules 151)
@@
     (descr "CuK sub miniature slide switch, JS series, DPDT, right angle, http://www.ckswitches.com/media/1422/js.pdf")
     (tags "switch DPDT")
-    (fp_text reference SW1 (at 0 -2 90) (layer F.SilkS)
+    (fp_text reference SW1 (at -1 5.05 270) (layer F.SilkS)
       (effects (font (size 1 1) (thickness 0.15)))
     )
@@
     )
   )
-  (gr_text 2018 (at 196.25 126.75) (layer F.SilkS)
+  (gr_text V1.0 (at 197 128.5) (layer F.SilkS)
+    (effects (font (size 1.5 1.5) (thickness 0.3)))
+  )
+  (gr_text 2018 (at 197.25 130.75) (layer F.SilkS)
     (effects (font (size 1.5 1.5) (thickness 0.3)))
   )
@@
   (gr_line (start 189.25 74) (end 190 73) (layer F.SilkS) (width 0.3))
   (gr_line (start 189.25 73) (end 190 74) (layer F.SilkS) (width 0.3))
-  (gr_circle (center 196.302775 129.5) (end 197.802775 130.5) (layer F.SilkS) (width 0.3))
-  (gr_text CC (at 196.25 129.5) (layer F.SilkS)
+  (gr_circle (center 197.5 124.697225) (end 199 125.697225) (layer F.SilkS) (width 0.3))
+  (gr_text CC (at 197.5 124.75) (layer F.SilkS)
     (effects (font (size 1.5 1.5) (thickness 0.3)))
   )
@@
   (via (at 150.17 130.08) (size 0.6) (drill 0.4) (layers F.Cu B.Cu) (net 16))
   (segment (start 147 130.08) (end 150.17 130.08) (width 0.25) (layer B.Cu) (net 16))
+  (segment (start 165 121.3) (end 166.3 121.3) (width 0.45) (layer F.Cu) (net 17))
+  (segment (start 167 122) (end 167 125.25) (width 0.45) (layer F.Cu) (net 17))
+  (segment (start 166.3 121.3) (end 167 122) (width 0.45) (layer F.Cu) (net 17))
+  (segment (start 167 125.25) (end 167.25 125.5) (width 0.45) (layer F.Cu) (net 17))
+  (segment (start 193.75 125.5) (end 195.25 127) (width 0.45) (layer F.Cu) (net 17))
+  (segment (start 167.25 125.5) (end 193.75 125.5) (width 0.45) (layer F.Cu) (net 17))
+  (segment (start 195.25 127) (end 200.5 127) (width 0.45) (layer F.Cu) (net 17))
   (segment (start 150.25 121.25) (end 149.25 121.25) (width 0.25) (layer F.Cu) (net 17))
   (segment (start 149.25 121.25) (end 149 121.5) (width 0.25) (layer F.Cu) (net 17))
@@
   (segment (start 187.5 131.5) (end 156.75 131.5) (width 0.25) (layer F.Cu) (net 17))
   (segment (start 188.45 130) (end 188.45 130.55) (width 0.25) (layer F.Cu) (net 17))
-  (segment (start 165 121.3) (end 166.3 121.3) (width 0.45) (layer F.Cu) (net 17))
-  (segment (start 166.3 121.3) (end 167 122) (width 0.45) (layer F.Cu) (net 17))
-  (segment (start 167 122) (end 167 125.25) (width 0.45) (layer F.Cu) (net 17))
-  (segment (start 167 125.25) (end 167.25 125.5) (width 0.45) (layer F.Cu) (net 17))
-  (segment (start 167.25 125.5) (end 199 125.5) (width 0.45) (layer F.Cu) (net 17))
-  (segment (start 199 125.5) (end 200.5 127) (width 0.45) (layer F.Cu) (net 17))
   (segment (start 177.75 106.2) (end 177.8 106.25) (width 0.45) (layer F.Cu) (net 17))
   (segment (start 177.8 106.25) (end 200.75 106.25) (width 0.45) (layer F.Cu) (net 17))
