File: hardware/Noise Meter.sch (KiCad schematic (older format))
At the start: 47 parts, among them J1 Conn_01x02, Q1 MMBT2222A, Q2 MMBT2222A, Q3 MMBT2222A, Q4 MMBT2222A, SW1 SW_DPST, U1 ISL28290, U2 LT6231, U3 AD8436, U4 PIC16F19156, U5 LCD-4-digit

Commit message: ready for pcb layout
Parts:
- removed C15: 10uF, symbol CP1
- removed C16: 3.3uF, symbol CP1
- removed J1: Conn_01x02, symbol Conn_01x02
- added C15, C16, C21: 22uF 20% 6.3V, Noise Meter Kicad Footprint Library:Feedthrough_C_0805_HandSoldering, symbol C_Feedthrough
- added C20: 1000uF, Capacitors_SMD:CP_Elec_10x10.5, symbol CP1
- added D1: 1N4148, Diodes_SMD:D_SOD-123, symbol D_Small_ALT
- added J1: Conn_Coaxial, Connectors_Molex:Molex_SMA_Jack_Edge_Mount, symbol Conn_Coaxial
- added J2: Conn_01x05_Male, Pin_Headers:Pin_Header_Angled_1x05_Pitch2.54mm, symbol Conn_01x05_Male
- added R16: 15K, Resistors_SMD:R_0603_HandSoldering, symbol R
- C1, C2: footprint (none) -> Capacitors_SMD:CP_Elec_4x4.5; Digikey P/N (none) -> Digikey P/N: PCE4527CT-ND; Manufacturer (none) -> Panasonic; Manufacturer P/N (none) -> EEE-FP1C100AR; Size (none) -> Dia.=4, L=4.3, H=5.8(mm); Size Code (none) -> Size B; Tolerance (none) -> +/-20%; Voltage (none) -> 16VDC
- C10, C11, C12, C13, C19, C3, C4, C6, C7: footprint (none) -> Capacitors_SMD:C_0603_HandSoldering
- C14: value 10uF -> 100uF; footprint (none) -> Capacitors_SMD:CP_Elec_6.3x7.7; Digikey P/N (none) -> Digikey P/N: PCE4533CT-ND; Manufacturer (none) -> Panasonic; Manufacturer P/N (none) -> EEE-FP1C101AP; Size (none) -> Dia.=6.3, L=6.6,H=5.8(mm); Size Code (none) -> Size D; Tolerance (none) -> +/-20%; Voltage (none) -> 16VDC
- C17: footprint (none) -> Capacitors_THT:C_Rect_L26.5mm_W8.5mm_P22.50mm_MKS4; Digikey P/N (none) -> Digikey P/N: 399-11495-ND; Manufacturer (none) -> KEMET; Manufacturer P/N (none) -> R60DN51005030J; Size (none) -> LWHS(mm)=26x8.5x17x22.5; Tolerance (none) -> 5%; Voltage (none) -> 63VDC
- C18: footprint (none) -> Capacitors_THT:C_Disc_D7.0mm_W2.5mm_P5.00mm; Digikey P/N (none) -> Digikey P/N: 399-5444-3-ND; Manufacturer (none) -> KEMET; Mnaufacturer P/N (none) -> R82DC3100DQ50J; Size (none) -> LWHS(mm)=7.2x2.5x6.6x5.0; Tolerance (none) -> 5%; Voltage (none) -> 63VDC
- C5: footprint (none) -> Capacitors_THT:C_Rect_L41.5mm_W24.0mm_P37.50mm_MKS4; Digikey P/N (none) -> Digikey P/N: 399-13010-ND; Manufacturer (none) -> KEMET; Manufacturer P/N (none) -> R60EW61005000K; Size (none) -> LWHS(mm)=41.5x24x44x37.5; Tolerance (none) -> 10%; Voltage (none) -> 100VDC
- C8: value CP1 -> 1000uF; footprint (none) -> Capacitors_SMD:CP_Elec_10x10.5; Digikey P/N (none) -> PCE4567CT-ND; Manufacturer (none) -> Panasonic; Manufacturer P/N (none) -> EEE-1AA102UAP; Size Code (none) -> Size G; Szie (none) -> L=10.2, Dia.10 (mm); Tolerance (none) -> +/-20%; Voltage (none) -> 10VDC
- C9: value CP1 -> 10uF; footprint (none) -> Capacitors_THT:C_Rect_L26.5mm_W8.5mm_P22.50mm_MKS4; Digikey P/N (none) -> Digikey P/N: 399-11495-ND; Manufacturer (none) -> KEMET; Manufacturer P/N (none) -> R60DN51005030J; Size (none) -> LWHS(mm)=26x8.5x17x22.5; Tolerance (none) -> 5%; Voltage (none) -> 63VDC
- R1, R10, R11, R12, R13, R14, R15, R3, R7, R8, R9: footprint (none) -> Resistors_SMD:R_0603_HandSoldering
- R2, R4: value 22 -> 24; footprint (none) -> Resistors_SMD:R_0603_HandSoldering
- R5: value 560 -> 680; footprint (none) -> Resistors_SMD:R_0603_HandSoldering
- R6: footprint (none) -> Potentiometers:Potentiometer_Trimmer_Bourns_3214J; Digikey P/N (none) -> 3214J-101ECT-ND; Manufacturer (none) -> Bourns; Manufacturer P/N (none) -> 3214J-1-101E
- U1: footprint (none) -> SMD_Packages:SOIC-8-N
Connections:
- net labels added: +3V_Digital, -3V_Digital
- wire segments 174 -> 152
Other:
- note added: "Alt. (Low ESR) EEE-FP1A102AP / PCE4434CT-ND"
- note added: "C1, C2"
- note added: "C14"
- note added: "C15, C16"
- note added: "C17"
- note added: "C18"
- note added: "C21"
- note added: "C5"
- note added: "C8"
- note added: "C9"
- note added: "R6"
- moved on the sheet: BT1, BT2, C14, C17, C18, C19, C3, C4, C5, C6, C7, C8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

Commit message: PCB V1.0
Parts:
- removed U1: ISL28290, SMD_Packages:SOIC-8-N, symbol ISL28290
- removed U2: LT6231, SMD_Packages:SOIC-8-N, symbol LT6231
- removed U5: LCD-4-digit, Connectors_Molex:Molex_MicroLatch-53253-1270_12x2.00mm_Straight, symbol LCD-4-digit
- added C1, C10, C2, C29, C3, C4, C6, C7, C8: 100uF, Capacitors_Tantalum_SMD:CP_Tantalum_Case-X_EIA-7343-43_Hand, symbol CP1
- added C31: 10uF, Capacitors_THT:C_Rect_L31.5mm_W13.0mm_P27.50mm_MKS4, symbol CP1
- added C33: 100nF, Capacitors_SMD:C_0603_HandSoldering, symbol C
- added CON1: LCD-4-digit, Noise Meter Kicad Footprint Library:4-digit-LCD-footprint, symbol LCD-4-digit
- added CON2: 5110_LCD, Noise Meter Kicad Footprint Library:5110, symbol 5110_LCD
- added CON3: 5110_LCD_ALT, Noise Meter Kicad Footprint Library:5110-Alt, symbol 5110_LCD_ALT
- added J3: Conn_01x02, Pin_Headers:Pin_Header_Angled_1x02_Pitch2.54mm, symbol Conn_01x02
- added L1, L2: FB, Inductors_SMD:L_0805, symbol L_Core_Ferrite_Small
- added R1: 15K, Resistors_SMD:R_0603_HandSoldering, symbol R
- added R2: 82, Resistors_SMD:R_0603_HandSoldering, symbol R
- added SW2, SW3, SW4, SW5: SW_Push, Buttons_Switches_SMD:SW_SPST_B3SL-1002P, symbol SW_Push
- added U1, U2: OPA2227EP, SMD_Packages:SOIC-8-N, symbol OPA2227EP
- C14: value 100uF -> 10uF; footprint Capacitors_SMD:CP_Elec_6.3x7.7 -> Capacitors_SMD:CP_Elec_4x4.5; Digikey P/N Digikey P/N: PCE4533CT-ND -> Digikey P/N: PCE4527CT-ND; Manufacturer P/N EEE-FP1C101AP -> EEE-FP1C100AR; Size Dia.=6.3, L=6.6,H=5.8(mm) -> Dia.=4, L=4.3, H=5.8(mm); Size Code Size D -> Size B
- C27: renamed from C17; footprint Capacitors_THT:C_Rect_L26.5mm_W8.5mm_P22.50mm_MKS4 -> Capacitors_THT:C_Rect_L31.5mm_W13.0mm_P27.50mm_MKS4; Digikey P/N Digikey P/N: 399-11495-ND -> Digikey P/N: 399-15654-ND; Manufacturer P/N R60DN51005030J -> C4AEGBU5100A1XK; Size LWHS(mm)=26x8.5x17x22.5 -> LBHS(mm)=31.5x13x25x27.5; Tolerance 5% -> 10%; Voltage 63VDC -> 450VDC
- C28: renamed from C18; footprint Capacitors_THT:C_Disc_D7.0mm_W2.5mm_P5.00mm -> Capacitors_THT:C_Rect_L13.0mm_W6.0mm_P10.00mm_FKS3_FKP3_MKS4; Digikey P/N Digikey P/N: 399-5444-3-ND -> (none); Manufacturer KEMET -> ECPOS/TDK; Mnaufacturer P/N R82DC3100DQ50J -> B32921C3104M000; Size LWHS(mm)=7.2x2.5x6.6x5.0 -> LWHS(mm)=13x6x12x10; Vendor P/N (none) -> RS P/N: 882-9477; Voltage 63VDC -> 305VAC
- C30: renamed from C21; value 22uF 20% 6.3V -> 0.1uF 20% 6.3V
- C5: footprint Capacitors_THT:C_Rect_L41.5mm_W24.0mm_P37.50mm_MKS4 -> Capacitors_Tantalum_SMD:CP_Tantalum_Case-X_EIA-7343-43_Hand; Digikey P/N Digikey P/N: 399-13010-ND -> 399-8410-1-ND; EIA Case Code (none) -> 7343-43; Manufacturer P/N R60EW61005000K -> T491X107K025AT; Size LWHS(mm)=41.5x24x44x37.5 -> (none); Size Code (none) -> Case X; Voltage 100VDC -> 25VDC
- C9: value 10uF -> 100uF; footprint Capacitors_THT:C_Rect_L26.5mm_W8.5mm_P22.50mm_MKS4 -> Capacitors_Tantalum_SMD:CP_Tantalum_Case-X_EIA-7343-43_Hand; Digikey P/N Digikey P/N: 399-11495-ND -> 399-8410-1-ND; EIA Case Code (none) -> 7343-43; Manufacturer P/N R60DN51005030J -> T491X107K025AT; Size LWHS(mm)=26x8.5x17x22.5 -> (none); Size Code (none) -> Case X; Tolerance 5% -> 10%; Voltage 63VDC -> 25VDC
- J1: footprint Connectors_Molex:Molex_SMA_Jack_Edge_Mount -> Noise Meter Kicad Footprint Library:SMA-CONN
- R3: renamed from R1; value 2.2K -> 510
- SW1: footprint Buttons_Switches_THT:SW_E-Switch_EG2219_DPDT_Angled -> Buttons_Switches_THT:SW_CuK_JS202011AQN_DPDT_Angled
- renumbered C13 to C12, C10 to C15, C12 to C16, C1 to C17, C3 to C18, C6 to C19, C2 to C20, C4 to C21, C7 to C22, C8 to C23, C20 to C24, C15 to C25, C16 to C26, C19 to C32, R5 to R10, R10 to R11, R14 to R12, R2 to R13, R4 to R14, R9 to R15, R13 to R16, R16 to R17, R15 to R18, R7 to R4, R8 to R5, R11 to R6, R12 to R7, R6 to R8, R3 to R9, U4 to U3, U3 to U5
Connections:
- net labels added: +3V_LNA, -3V_LNA
- wire segments 152 -> 244
- no-connect marks 8 -> 11
Other:
- note added: "C1 - C10"
- note added: "C14/R1 provisional remedy for\n high output offset voltages."
- note added: "C17, C20"
- note added: "C23"
- note added: "C24"
- note added: "C25, C26"
- note added: "C27"
- note added: "C28"
- note added: "C29"
- note added: "C30"
- note added: "C31"
- note added: "R7"
- note added: "http://www.hkepc.com/forum/viewthread.php?fid=146&tid=2419038&extra=page%3D1"
- note removed: "C1, C2"
- note removed: "C14"
- note removed: "C15, C16"
- note removed: "C17"
- note removed: "C18"
- note removed: "C21"
- note removed: "C5"
- note removed: "C8"
- note removed: "C9"
- note removed: "R6"
- moved on the sheet: BT1, BT2, C11, C12, C18, C19, C21, C22, C32, D1, J1, J2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

Commit message: final touch ups and gerber files added
Connections:
- net Vrms: now reaches C30.1, J3.1 (Pin_1), U3.10 (SEG6/RA6)
Changed lines of the file:
@@
 $EndComp
 Connection ~ 4050 5950
+Text Label 4400 5650 0    60   ~ 0
+Vrms
 $EndSCHEMATC
